File: pcb/dut.kicad_sch (KiCad schematic)
At the start: 0 parts

Commit message: dut components update
Parts:
- added DUT1: ~, Package_QFP:TQFP-144_20x20mm_P0.5mm, symbol dut:dut_tqfp144
Changed lines of the file:
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@@
 	(generator_version "9.0")
 	(paper "A4")
+	(symbol
+		(lib_id "dut:dut_tqfp144")
+		(at 135.89 85.09 0)
+		(unit 1)
+		(exclude_from_sim no)
+		(in_bom yes)
+		(on_board yes)
+		(dnp no)
+		(fields_autoplaced yes)
+		(property "Reference" "DUT1"
+			(at 164.7033 123.19 0)
+			(effects
+				(font
+					(size 1.27 1.27)
+				)
+				(justify left)
+			)
+		)
+		(property "Value" "~"
+			(at 164.7033 124.46 0)
+			(effects
+				(font
+					(size 1.27 1.27)
+				)
+				(justify left)
+			)
+		)
+		(property "Footprint" "Package_QFP:TQFP-144_20x20mm_P0.5mm"
+			(at 135.89 85.09 0)
+			(effects
+				(font
+					(size 1.27 1.27)
+				)
+				(hide yes)
+			)
+		)
+		(property "Datasheet" ""
+			(at 135.89 85.09 0)
+			(effects
+				(font
+					(size 1.27 1.27)
+				)
+				(hide yes)
+			)
+		)
+		(property "Description" ""
+			(at 135.89 85.09 0)
+			(effects
+				(font
+					(size 1.27 1.27)
+				)
+				(hide yes)
+			)
+		)
+		(pin "9"
+		)
+		(pin "11"
+		)
+		(pin "15"
+		)
+		(pin "12"
+		)
+		(pin "4"
+		)
+		(pin "6"
+		)
+		(pin "7"
+		)
+		(pin "13"
+		)
+		(pin "1"
+		)
+		(pin "2"
+		)
+		(pin "3"
+		)
+		(pin "5"
+		)
+		(pin "8"
+		)
+		(pin "10"
+		)
+		(pin "14"
+		)
+		(pin "36"
+		)
+		(pin "22"
+		)
+		(pin "26"
+		)
+		(pin "30"
+		)
+		(pin "23"
+		)
+		(pin "16"
+		)
+		(pin "17"
+		)
+		(pin "18"
+		)
+		(pin "19"
+		)
+		(pin "21"
+		)
+		(pin "34"
+		)
+		(pin "31"
+		)
+		(pin "33"
+		)
+		(pin "32"
+		)
+		(pin "20"
+		)
+		(pin "27"
+		)
+		(pin "24"
+		)
+		(pin "35"
+		)
+		(pin "25"
+		)
+		(pin "28"
+		)
+		(pin "29"
+		)
+		(instances
+			(project ""
+				(path "/1a761ede-a9cd-4cca-ba56-e59a7a4d7b19/15b02fdd-7eee-4532-93a1-61532bb4dec6"
+					(reference "DUT1")
+					(unit 1)
+				)
+			)
+		)
+	)
 )
