File: pcb/pll.kicad_sch (KiCad schematic)
At the start: 0 parts

Commit message: DAC/JTAG updates
Other:
- sheet DACAnalogswitch ports: added DAC0, DAC1, DAC2, DAC3, VDD, VIO; removed none
Changed lines of the file:
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@@
 	(paper "A4")
+	(junction
+		(at 144.78 69.85)
+		(diameter 0)
+		(color 0 0 0 0)
+	)
 	(junction
 		(at 80.01 77.47)
@@
 	)
 	(junction
+		(at 124.46 69.85)
+		(diameter 0)
+		(color 0 0 0 0)
+	)
+	(junction
 		(at 77.47 83.82)
 		(diameter 0)
@@
 	(wire
 		(pts
+			(xy 144.78 64.77) (xy 147.32 64.77)
+		)
+		(stroke
+			(width 0)
+			(type default)
+		)
+	)
+	(wire
+		(pts
 			(xy 52.07 96.52) (xy 52.07 88.9)
 		)
@@
 	(wire
 		(pts
-			(xy 138.43 81.28) (xy 138.43 76.2)
+			(xy 130.81 48.26) (xy 130.81 86.36)
 		)
 		(stroke
@@
 	(wire
 		(pts
-			(xy 142.24 76.2) (xy 142.24 83.82)
-		)
-		(stroke
-			(width 0)
-			(type default)
-		)
-	)
-	(wire
-		(pts
-			(xy 130.81 76.2) (xy 130.81 86.36)
+			(xy 138.43 44.45) (xy 138.43 86.36)
+		)
+		(stroke
+			(width 0)
+			(type default)
+		)
+	)
+	(wire
+		(pts
+			(xy 127 44.45) (xy 127 48.26)
 		)
 		(stroke
@@
 	(wire
 		(pts
-			(xy 124.46 76.2) (xy 124.46 86.36)
-		)
-		(stroke
-			(width 0)
-			(type default)
-		)
-	)
-	(wire
-		(pts
-			(xy 138.43 83.82) (xy 138.43 86.36)
+			(xy 144.78 69.85) (xy 144.78 64.77)
+		)
+		(stroke
+			(width 0)
+			(type default)
+		)
+	)
+	(wire
+		(pts
+			(xy 124.46 69.85) (xy 124.46 86.36)
+		)
+		(stroke
+			(width 0)
+			(type default)
+		)
+	)
+	(wire
+		(pts
+			(xy 120.65 44.45) (xy 120.65 49.53)
+		)
+		(stroke
+			(width 0)
+			(type default)
+		)
+	)
+	(wire
+		(pts
+			(xy 127 48.26) (xy 130.81 48.26)
+		)
+		(stroke
+			(width 0)
+			(type default)
+		)
+	)
+	(wire
+		(pts
+			(xy 124.46 69.85) (xy 144.78 69.85)
+		)
+		(stroke
+			(width 0)
+			(type default)
+		)
+	)
+	(wire
+		(pts
+			(xy 120.65 49.53) (xy 124.46 49.53)
 		)
 		(stroke
@@
 	(wire
 		(pts
-			(xy 134.62 86.36) (xy 134.62 81.28)
+			(xy 134.62 44.45) (xy 134.62 86.36)
 		)
 		(stroke
@@
 	(wire
 		(pts
+			(xy 144.78 69.85) (xy 147.32 69.85)
+		)
+		(stroke
+			(width 0)
+			(type default)
+		)
+	)
+	(wire
+		(pts
 			(xy 77.47 83.82) (xy 80.01 83.82)
 		)
@@
 	(wire
 		(pts
+			(xy 124.46 49.53) (xy 124.46 69.85)
+		)
+		(stroke
+			(width 0)
+			(type default)
+		)
+	)
+	(wire
+		(pts
 			(xy 90.17 80.01) (xy 90.17 76.2)
 		)
@@
 		(pts
 			(xy 74.93 83.82) (xy 71.12 83.82)
-		)
-		(stroke
-			(width 0)
-			(type default)
-		)
-	)
-	(wire
-		(pts
-			(xy 134.62 81.28) (xy 138.43 81.28)
-		)
-		(stroke
-			(width 0)
-			(type default)
-		)
-	)
-	(wire
-		(pts
-			(xy 142.24 83.82) (xy 138.43 83.82)
 		)
 		(stroke
@@
 	)
 	(sheet
-		(at 119.38 55.88)
+		(at 115.57 24.13)
 		(size 49.53 20.32)
 		(exclude_from_sim no)
@@
 		)
 		(property "Sheetname" "usb-serial"
-			(at 119.38 55.1684 0)
+			(at 115.57 23.4184 0)
 			(effects
 				(font
@@
 		)
 		(property "Sheetfile" "usb-serial.kicad_sch"
-			(at 119.38 76.7846 0)
+			(at 115.57 45.0346 0)
 			(effects
 				(font
@@
 		)
 		(pin "VDD" input
-			(at 124.46 76.2 270)
+			(at 120.65 44.45 270)
 			(effects
 				(font
@@
 		)
 		(pin "VBUS" input
-			(at 130.81 76.2 270)
+			(at 127 44.45 270)
 			(effects
 				(font
@@
 		)
 		(pin "D-" input
-			(at 138.43 76.2 270)
+			(at 134.62 44.45 270)
 			(effects
 				(font
@@
 		)
 		(pin "D+" input
-			(at 142.24 76.2 270)
+			(at 138.43 44.45 270)
 			(effects
 				(font
@@
 	)
 	(sheet
-		(at 217.17 109.22)
+		(at 147.32 59.69)
 		(size 38.1 22.86)
 		(exclude_from_sim no)
@@
 		)
 		(property "Sheetname" "DACAnalogswitch"
-			(at 217.17 108.5084 0)
+			(at 147.32 58.9784 0)
 			(effects
 				(font
@@
 		)
 		(property "Sheetfile" "dac_switch.kicad_sch"
-			(at 217.17 132.6646 0)
+			(at 147.32 83.1346 0)
 			(effects
 				(font
@@
 			)
 		)
+		(pin "VDD" input
+			(at 147.32 64.77 180)
+			(effects
+				(font
+					(size 1.27 1.27)
+				)
+				(justify left)
+			)
+		)
+		(pin "VIO" input
+			(at 147.32 69.85 180)
+			(effects
+				(font
+					(size 1.27 1.27)
+				)
+				(justify left)
+			)
+		)
+		(pin "DAC0" output
+			(at 185.42 63.5 0)
+			(effects
+				(font
+					(size 1.27 1.27)
+				)
+				(justify right)
+			)
+		)
+		(pin "DAC1" output
+			(at 185.42 67.31 0)
+			(effects
+				(font
+					(size 1.27 1.27)
+				)
+				(justify right)
+			)
+		)
+		(pin "DAC3" output
+			(at 185.42 74.93 0)
+			(effects
+				(font
+					(size 1.27 1.27)
+				)
+				(justify right)
+			)
+		)
+		(pin "DAC2" output
+			(at 185.42 71.12 0)
+			(effects
+				(font
+					(size 1.27 1.27)
+				)
+				(justify right)
+			)
+		)
