File: pcb/fpga.kicad_sch (KiCad schematic)
At the start: 15 parts, among them J1 6pin_2mm_jtag, U1 XC6SLX4-TQG144, U2 AT45DB161-JC, Y1 DSC1004AL1-001.0000

Commit message: external crystal
Parts:
- added C44: 0.1uF, Capacitor_SMD:C_0402_1005Metric, symbol Device:C
- added C46: 15pF, Capacitor_SMD:C_0402_1005Metric, symbol Device:C
Connections:
- net VCCOAUX is gone; now on net VCCAUX: J1.6 (VDD)
- net GND: now also Y1.2 (GND), C44.2, C46.2
- net VCCAUX: now also Y1.1 (~{STANDBY}), Y1.4 (VDD), C44.1
- net EXT_CLOCK: now reaches Y1.3 (OUT)
- net EXT_CLOCK: now also U1.55 (IO_L30N_GCLK0_USERCCLK_2), C46.1
Other:
- moved on the sheet: Y1
