File: pcb/dac_switch.kicad_sch (KiCad schematic)
At the start: 1 part, among them U5 DAC80504

Commit message: DAC/JTAG updates
Parts:
- added C47, C48, C49, C50: 0.1uF, Capacitor_SMD:C_0402_1005Metric, symbol Device:C
Connections:
- net GND: now reaches U5.10 (REFDIV)
- net GND: now also U5.11 (~{LDAC}), U5.17 (EP), U5.6 (GND), U5.9 (RSTSEL), C47.2, C48.2, C49.2, C50.2
- net VIO: now reaches U5.16 (VIO)
- net VIO: now also U5.8 (GAIN), C49.1, C50.1
- net DAC0: now reaches U5.2 (OUT0)
- net DAC1: now reaches U5.3 (OUT1)
- net DAC2: now reaches U5.4 (OUT2)
- net DAC3: now reaches U5.5 (OUT3)
- net VDD: now reaches U5.7 (VDD)
- net VDD: now also C47.1, C48.1
