File: pcb/pll.kicad_pcb (KiCad board)
At the start: 4 copper layers, 205.8 x 90.1 mm, 75 parts, among them J1 6pin_2mm_jtag, J2 USB3090-XX-X_REVE2, U1 XC6SLX4-TQG144, U2 AT45DB161-JC, U3 CP2102N-A01-GQFN28, U4 TPS650250RHBR, U5 DAC80504, Y1 DSC1004AL1-001.0000

Commit message: dut components update
Parts:
- added DUT1: ~, Package_QFP:TQFP-144_20x20mm_P0.5mm, F.Cu at (160.2, 85.0)
- added J5: 85_SMA-50-0-144_111_YE, coax_connector:HUBER_SUHNER_85_SMA-50-0-144_111_YE, F.Cu at (194.0, 39.1)
- added J6: 85_SMA-50-0-144_111_YE, coax_connector:HUBER_SUHNER_85_SMA-50-0-144_111_YE, F.Cu at (237.9, 62.1)
- added J7: 85_SMA-50-0-144_111_YE, coax_connector:HUBER_SUHNER_85_SMA-50-0-144_111_YE, F.Cu at (195.3, 115.1)
- added J8: 85_SMA-50-0-144_111_YE, coax_connector:HUBER_SUHNER_85_SMA-50-0-144_111_YE, F.Cu at (236.8, 85.5)
- added T1: ~, TIA:QFN50P300X300X80-16N, F.Cu at (194.9, 82.9)
Routing:
- net (no net): track 2.64 -> 1.88 mm

Commit message: external crystal
Parts:
- added C44: 0.1uF, Capacitor_SMD:C_0402_1005Metric, B.Cu at (103.6, 104.0)
- added C46: 15pF, Capacitor_SMD:C_0402_1005Metric, B.Cu at (108.8, 103.8)
- moved S2 11.8 mm to (86.2, 111.8)
- moved J5 11.5 mm to (192.6, 50.5), turned to 180 degrees
- moved J6 10.1 mm to (228.6, 65.9), turned to 90 degrees
- moved J8 8.45 mm to (228.4, 84.2), turned to 90 degrees
- moved DUT1 8.36 mm to (161.6, 76.8)
- moved J7 6.69 mm to (193.2, 108.7), turned to 0 degrees
- moved C14 2.02 mm to (109.0, 96.8), turned to 180 degrees
- moved Y1 1.74 mm to (106.2, 108.5), turned to 90 degrees
Connections:
- J1 pad 6: /fpga/VCCOAUX -> /fpga/VCCAUX
- U1 pad 55: unconnected-(U1B-IO_L30N_GCLK0_USERCCLK_2-Pad55) -> /fpga/EXT_CLOCK
- Y1 pad 1: unconnected-(Y1-~{STANDBY}-Pad1) -> /fpga/VCCAUX
- Y1 pad 2: unconnected-(Y1-GND-Pad2) -> GND
- Y1 pad 3: unconnected-(Y1-OUT-Pad3) -> /fpga/EXT_CLOCK
- Y1 pad 4: unconnected-(Y1-VDD-Pad4) -> /fpga/VCCAUX
Routing:
- net /fpga/VCCAUX: track 266.2 -> 308.5 mm, vias 28 -> 29
- net /fpga/EXT_CLOCK: track 0.00 -> 14.7 mm, vias 0 -> 1
- net /fpga/PROG_B: track 21.2 -> 29.5 mm
- net GND: track 99.0 -> 100.8 mm, vias 57 -> 60
- net (no net): track 1.88 -> 0.00 mm

Commit message: DAC/JTAG updates
Parts:
- added C47: 0.1uF, Capacitor_SMD:C_0402_1005Metric, B.Cu at (140.2, 76.5)
- added C48: 0.1uF, Capacitor_SMD:C_0402_1005Metric, B.Cu at (141.3, 76.5)
- added C49: 0.1uF, Capacitor_SMD:C_0402_1005Metric, B.Cu at (134.3, 78.5)
- added C50: 0.1uF, Capacitor_SMD:C_0402_1005Metric, B.Cu at (138.6, 73.8)
- moved DUT1 17.8 mm to (179.1, 80.2)
- moved T1 15.8 mm to (210.0, 77.9), turned to -90 degrees
- moved U5 8.74 mm to (137.1, 77.2), turned to 90 degrees
- moved C5 5.42 mm to (126.0, 95.4), turned to 0 degrees
- moved D3 3.22 mm to (127.2, 99.2)
- moved R13 2.19 mm to (126.5, 102.9)
- moved C21 0.69 mm to (124.5, 78.0), turned to 0 degrees
Connections:
- C37 pad 1: /power/VLDO1 -> /DACAnalogswitch/VDD
- C38 pad 1: /power/VLDO1 -> /DACAnalogswitch/VDD
- C45 pad 1: /power/VLDO1 -> /DACAnalogswitch/VDD
- R11 pad 1: /power/VLDO1 -> /DACAnalogswitch/VDD
- R12 pad 1: /power/VLDO1 -> /DACAnalogswitch/VDD
- U3 pad 6: /power/VLDO1 -> /DACAnalogswitch/VDD
- U4 pad 16: /power/VLDO1 -> /DACAnalogswitch/VDD
- U4 pad 33: unconnected-(U4-EP-Pad33) -> GND
- U5 pad 10: unconnected-(U5-REFDIV-Pad10) -> GND
- U5 pad 11: unconnected-(U5-~{LDAC}-Pad11) -> GND
- U5 pad 16: unconnected-(U5-VIO-Pad16) -> /DACAnalogswitch/VDD
- U5 pad 17: unconnected-(U5-EP-Pad17) -> GND
- U5 pad 2: unconnected-(U5-OUT0-Pad2) -> /DACAnalogswitch/DAC0
- U5 pad 3: unconnected-(U5-OUT1-Pad3) -> /DACAnalogswitch/DAC1
- U5 pad 4: unconnected-(U5-OUT2-Pad4) -> /DACAnalogswitch/DAC2
- U5 pad 5: unconnected-(U5-OUT3-Pad5) -> /DACAnalogswitch/DAC3
- U5 pad 6: unconnected-(U5-GND-Pad6) -> GND
- U5 pad 7: unconnected-(U5-VDD-Pad7) -> /DACAnalogswitch/VDD
- U5 pad 8: unconnected-(U5-GAIN-Pad8) -> /DACAnalogswitch/VDD
- U5 pad 9: unconnected-(U5-RSTSEL-Pad9) -> GND
Routing:
- net /DACAnalogswitch/VDD: track 0.00 -> 154.6 mm, vias 0 -> 5
- net /power/VLDO1: track 81.6 -> 0.00 mm, vias 2 -> 0
- net /fpga/VCCAUX: track 308.5 -> 312.3 mm, vias 29 -> 30
- net /fpga/DONE: track 13.1 -> 10.1 mm
- net /fpga/VCCINT: track 97.8 -> 100.4 mm
- net /fpga/TCK: track 16.2 -> 14.6 mm, vias 1 -> 0
- net GND: track 100.8 -> 101.8 mm, vias 60 -> 63
- net /fpga/TDI: track 16.1 -> 17.0 mm
- net /fpga/TMS: track 37.0 -> 37.8 mm
- net /fpga/TDO: track 36.8 -> 37.4 mm
